Commit message: Fixed unstable URDF Gazebo

File: description/robot_core.xacro (robot description, xacro)
@@ -10,4 +10,5 @@
         <parent link="world"/>
         <child link="base_link"/>
+        <dynamics damping="1000000" friction="10000000"/>
     </joint>
     <!-- base_link is a large rectangular plate. Some things to note: -->
@@ -28,13 +29,8 @@
         <collision>
             <origin xyz="0 0 0.05" rpy="0 0 0"/>
-            <geometry>
-                <box size="0 0 0" />
-            </geometry>
-        </collision>
-        <inertial>
-            <origin xyz="0 0 0" rpy="0 0 0"/>
-            <mass value="10" />
-            <inertia ixx="0.01" ixy="0" ixz="0" iyy="0.01" iyz="0.0" izz="0.01" />
-        </inertial>
+        </collision>
+        <xacro:inertial_box mass="10" x="5" y="5" z="0.1">
+            <origin xyz="0 0 0.05" rpy="0 0 0"/>
+        </xacro:inertial_box>
     </link>
     <joint name="pilar1_joint" type="fixed">
@@ -42,4 +38,5 @@
         <parent link="base_link"/>
         <child link="pilar1_link"/>
+        <dynamics damping="1000000" friction="10000000"/>
     </joint>
     <link name="pilar1_link">
@@ -54,14 +51,9 @@
         </visual>
         <collision>
-            <origin xyz="0 0 0" rpy="0 0 0"/>
-            <geometry>
-                <box size="0.25 0.25 2" />
-            </geometry>
-        </collision>
-        <inertial>
-            <origin xyz="0 0 0" rpy="0 0 0"/>
-            <mass value="3" />
-            <inertia ixx="0.01" ixy="0" ixz="0" iyy="0.01" iyz="0.0" izz="0.01" />
-        </inertial>
+            <origin xyz="0 0 1" rpy="0 0 0"/>
+        </collision>
+        <xacro:inertial_box mass="2" x="0.5" y="0.25" z="0.15">
+            <origin xyz="0 0 1" rpy="0 0 0"/>
+        </xacro:inertial_box>
     </link>
     <joint name="pilar2_joint" type="fixed">
@@ -69,4 +61,5 @@
         <parent link="base_link"/>
         <child link="pilar2_link"/>
+        <dynamics damping="1000000" friction="10000000"/>
     </joint>
     <link name="pilar2_link">
@@ -81,14 +74,9 @@
         </visual>
         <collision>
-            <origin xyz="0 0 0" rpy="0 0 0"/>
-            <geometry>
-                <box size="0.25 0.25 2" />
-            </geometry>
-        </collision>
-        <inertial>
-            <origin xyz="0 0 0" rpy="0 0 0"/>
-            <mass value="3" />
-            <inertia ixx="0.01" ixy="0" ixz="0" iyy="0.01" iyz="0.0" izz="0.01" />
-        </inertial>
+            <origin xyz="0 0 1" rpy="0 0 0"/>
+        </collision>
+        <xacro:inertial_box mass="2" x="0.5" y="0.25" z="0.15">
+            <origin xyz="0 0 1" rpy="0 0 0"/>
+        </xacro:inertial_box>
     </link>
      <joint name="pilar3_joint" type="fixed">
@@ -96,4 +84,5 @@
         <parent link="base_link"/>
         <child link="pilar3_link"/>
+        <dynamics damping="1000000" friction="10000000"/>
     </joint>
     <link name="pilar3_link">
@@ -101,21 +90,15 @@
             <origin xyz="0 0 1" rpy="0 0 0"/>
             <geometry>
-                <box size="0.25 0.25 2" />
-            </geometry>
-            <material name="green">
-                <color rgba="0.2 1 0.2 1"/>
-            </material>
-        </visual>
-        <collision>
-            <origin xyz="0 0 0" rpy="0 0 0"/>
-            <geometry>
-                <box size="0.25 0.25 2" />
-            </geometry>
-        </collision>
-        <inertial>
-            <origin xyz="0 0 0" rpy="0 0 0"/>
-            <mass value="3" />
-            <inertia ixx="0.01" ixy="0" ixz="0" iyy="0.01" iyz="0.0" izz="0.01" />
-        </inertial>
+            </geometry>
+            <material name="green">
+                <color rgba="0.2 1 0.2 1"/>
+            </material>
+        </visual>
+        <collision>
+            <origin xyz="0 0 1" rpy="0 0 0"/>
+        </collision>
+        <xacro:inertial_box mass="2" x="0.5" y="0.25" z="0.15">
+            <origin xyz="0 0 1" rpy="0 0 0"/>
+        </xacro:inertial_box>
     </link>
     <joint name="pilar4_joint" type="fixed">
@@ -123,4 +106,5 @@
         <parent link="base_link"/>
         <child link="pilar4_link"/>
+        <dynamics damping="1000000" friction="10000000"/>
     </joint>
     <link name="pilar4_link">
@@ -135,14 +119,9 @@
         </visual>
         <collision>
-            <origin xyz="0 0 0" rpy="0 0 0"/>
-            <geometry>
-                <box size="0.25 0.25 2" />
-            </geometry>
-        </collision>
-        <inertial>
-            <origin xyz="0 0 0" rpy="0 0 0"/>
-            <mass value="3" />
-            <inertia ixx="0.01" ixy="0" ixz="0" iyy="0.01" iyz="0.0" izz="0.01" />
-        </inertial>
+            <origin xyz="0 0 1" rpy="0 0 0"/>
+        </collision>
+        <xacro:inertial_box mass="2" x="0.5" y="0.25" z="0.15">
+            <origin xyz="0 0 1" rpy="0 0 0"/>
+        </xacro:inertial_box>
     </link>
     <joint name="edge1_joint" type="fixed">
@@ -150,4 +129,5 @@
         <parent link="pilar1_link"/>
         <child link="edge1_link"/>
+        <dynamics damping="1000000" friction="10000000"/>
     </joint>
     <link name="edge1_link">
@@ -163,13 +143,8 @@
         <collision>
             <origin xyz="0 0 0" rpy="0 0 0"/>
-            <geometry>
-                <box size="0.25 2 0.25" />
-            </geometry>
-        </collision>
-        <inertial>
-            <origin xyz="0 0 0" rpy="0 0 0"/>
-            <mass value="3" />
-            <inertia ixx="0.01" ixy="0" ixz="0" iyy="0.01" iyz="0.0" izz="0.01" />
-        </inertial>
+        </collision>
+        <xacro:inertial_box mass="1" x="0.5" y="0.25" z="0.15">
+            <origin xyz="0 0 0.075" rpy="0 0 0"/>
+        </xacro:inertial_box>
     </link>
      <joint name="edge2_joint" type="fixed">
@@ -177,4 +152,5 @@
         <parent link="pilar2_link"/>
         <child link="edge2_link"/>
+        <dynamics damping="1000000" friction="10000000"/>
     </joint>
     <link name="edge2_link">
@@ -190,13 +166,8 @@
         <collision>
             <origin xyz="0 0 0" rpy="0 0 0"/>
-            <geometry>
-                <box size="0.25 2 0.25" />
-            </geometry>
-        </collision>
-        <inertial>
-            <origin xyz="0 0 0" rpy="0 0 0"/>
-            <mass value="3" />
-            <inertia ixx="0.01" ixy="0" ixz="0" iyy="0.01" iyz="0.0" izz="0.01" />
-        </inertial>
+        </collision>
+        <xacro:inertial_box mass="1" x="0.5" y="0.25" z="0.15">
+            <origin xyz="0 0 0" rpy="0 0 0"/>
+        </xacro:inertial_box>
     </link>
     <joint name="y_joint" type="prismatic">
@@ -219,14 +190,9 @@
         </visual>
         <collision>
-            <origin xyz="0 0 0" rpy="0 0 0"/>
-            <geometry>
-                <box size="4.5 0.25 0.25" />
-            </geometry>
-        </collision>
-        <inertial>
-            <origin xyz="0 0 0" rpy="0 0 0"/>
-            <mass value="2" />
-            <inertia ixx="0.01" ixy="0" ixz="0" iyy="0.01" iyz="0.0" izz="0.01" />
-        </inertial>
+            <origin xyz="2.25 0 0" rpy="0 0 0"/>
+        </collision>
+        <xacro:inertial_box mass="0.5" x="0.5" y="0.25" z="0.15">
+            <origin xyz="2.25 0 0" rpy="0 0 0"/>
+        </xacro:inertial_box>
     </link>
     <joint name="x_joint" type="prismatic">
@@ -249,14 +215,9 @@
         </visual>
         <collision>
-            <origin xyz="0 0 0" rpy="0 0 0"/>
-            <geometry>
-                <box size="0.25 0.25 1.5" />
-            </geometry>
-        </collision>
-        <inertial>
-            <origin xyz="0 0 0" rpy="0 0 0"/>
-            <mass value="1" />
-            <inertia ixx="0.01" ixy="0" ixz="0" iyy="0.01" iyz="0.0" izz="0.01" />
-        </inertial>
+            <origin xyz="0 0 -0.6" rpy="0 0 0"/>
+        </collision>
+        <xacro:inertial_box mass="0.5" x="0.5" y="0.25" z="0.15">
+            <origin xyz="0 0 -0.6" rpy="0 0 0"/>
+        </xacro:inertial_box>
     </link>
     <joint name="z_joint" type="prismatic">
@@ -277,14 +238,9 @@
         </visual>
         <collision>
-            <origin xyz="0 0 0" rpy="0 0 0"/>
-            <geometry>
-                <box size="0.25 0.25 0.4" />
-            </geometry>
-        </collision>
-        <inertial>
-            <origin xyz="0 0 0" rpy="0 0 0"/>
-            <mass value="0.5" />
-            <inertia ixx="0.01" ixy="0" ixz="0" iyy="0.01" iyz="0.0" izz="0.01" />
-        </inertial>
+            <origin xyz="0 0 -0.6" rpy="0 0 0"/>
+        </collision>
+        <xacro:inertial_box mass="0.2" x="0.5" y="0.25" z="0.15">
+            <origin xyz="0 0 -0.6" rpy="0 0 0"/>
+        </xacro:inertial_box>
     </link>
 </robot>

Commit message: trying to spawn the controller_managers

File: description/robot_core.xacro (robot description, xacro)
@@ -29,4 +29,7 @@
         <collision>
             <origin xyz="0 0 0.05" rpy="0 0 0"/>
+            <geometry>
+                <box size="5 5 0.1" />
+            </geometry>
         </collision>
         <xacro:inertial_box mass="10" x="5" y="5" z="0.1">
@@ -52,4 +55,7 @@
         <collision>
             <origin xyz="0 0 1" rpy="0 0 0"/>
+            <geometry>
+                <box size="0.25 0.25 2" />
+            </geometry>
         </collision>
         <xacro:inertial_box mass="2" x="0.5" y="0.25" z="0.15">
@@ -75,4 +81,7 @@
         <collision>
             <origin xyz="0 0 1" rpy="0 0 0"/>
+            <geometry>
+                <box size="0.25 0.25 2" />
+            </geometry>
         </collision>
         <xacro:inertial_box mass="2" x="0.5" y="0.25" z="0.15">
@@ -90,11 +99,15 @@
             <origin xyz="0 0 1" rpy="0 0 0"/>
             <geometry>
-            </geometry>
-            <material name="green">
-                <color rgba="0.2 1 0.2 1"/>
-            </material>
-        </visual>
-        <collision>
-            <origin xyz="0 0 1" rpy="0 0 0"/>
+                <box size="0.25 0.25 2" />
+            </geometry>
+            <material name="green">
+                <color rgba="0.2 1 0.2 1"/>
+            </material>
+        </visual>
+        <collision>
+            <origin xyz="0 0 1" rpy="0 0 0"/>
+            <geometry>
+                <box size="0.25 0.25 2" />
+            </geometry>
         </collision>
         <xacro:inertial_box mass="2" x="0.5" y="0.25" z="0.15">
@@ -120,4 +133,7 @@
         <collision>
             <origin xyz="0 0 1" rpy="0 0 0"/>
+            <geometry>
+                <box size="0.25 0.25 2" />
+            </geometry>
         </collision>
         <xacro:inertial_box mass="2" x="0.5" y="0.25" z="0.15">
@@ -143,4 +159,7 @@
         <collision>
             <origin xyz="0 0 0" rpy="0 0 0"/>
+            <geometry>
+                <box size="0.25 5 0.25" />
+            </geometry>
         </collision>
         <xacro:inertial_box mass="1" x="0.5" y="0.25" z="0.15">
@@ -166,4 +185,7 @@
         <collision>
             <origin xyz="0 0 0" rpy="0 0 0"/>
+            <geometry>
+                <box size="0.25 5 0.25" />
+            </geometry>
         </collision>
         <xacro:inertial_box mass="1" x="0.5" y="0.25" z="0.15">
@@ -191,4 +213,7 @@
         <collision>
             <origin xyz="2.25 0 0" rpy="0 0 0"/>
+            <geometry>
+                <box size="4.5 0.25 0.25" />
+            </geometry>
         </collision>
         <xacro:inertial_box mass="0.5" x="0.5" y="0.25" z="0.15">
@@ -216,4 +241,7 @@
         <collision>
             <origin xyz="0 0 -0.6" rpy="0 0 0"/>
+            <geometry>
+                <box size="0.25 0.25 1.75" />
+            </geometry>
         </collision>
         <xacro:inertial_box mass="0.5" x="0.5" y="0.25" z="0.15">
@@ -239,4 +267,7 @@
         <collision>
             <origin xyz="0 0 -0.6" rpy="0 0 0"/>
+            <geometry>
+                <box size="0.25 0.25 0.4" />
+            </geometry>
         </collision>
         <xacro:inertial_box mass="0.2" x="0.5" y="0.25" z="0.15">
