Commit message: fixed the gazebo parameters, inertial, collision, etc

File: description/example_gazebo.xacro (robot description, xacro)
@@ -9,23 +9,30 @@
         <material>Gazebo/Green</material>
     </gazebo>
-    <gazebo reference="slider_link">
+    <gazebo reference="x_link">
         <material>Gazebo/Blue</material>
     </gazebo>
-    <gazebo reference="arm_link">
+    <gazebo reference="y_link">
+        <material>Gazebo/Blue</material>
+    </gazebo>
+    <gazebo reference="z_link">
         <material>Gazebo/Orange</material>
     </gazebo>
     <!-- Gazebo requires the use of plugins to interact with other systems such as ROS. -->
-    <ros2_control name="GantrySystem" type="system">
-            <hardware>
-                <plugin>gazebo_ros2_control/GazeboSystem</plugin>
-            </hardware>
-            <joint name="slider_joint">
-                <command_interface name="position" />
-                <state_interface name="position" />
-            </joint>
-            <joint name="arm_joint">
-                <command_interface name="position" />
-                <state_interface name="position" />
-            </joint>
+    <ros2_control name="GazeboSystem" type="system">
+        <hardware>
+            <plugin>gazebo_ros2_control/GazeboSystem</plugin>
+        </hardware>
+        <joint name="x_joint">
+            <command_interface name="position" />
+            <state_interface name="position" />
+        </joint>
+        <joint name="y_joint">
+            <command_interface name="position" />
+            <state_interface name="position" />
+        </joint>
+        <joint name="z_joint">
+            <command_interface name="position" />
+            <state_interface name="position" />
+        </joint>
     </ros2_control>
     <gazebo>
@@ -34,69 +41,3 @@
         </plugin>
     </gazebo>
-    <!-- This plugin will publish the joint_states for the selected joints
-            (which robot_state_publisher can then use to broadcast the approprate tf). -->
-    <gazebo>
-        <plugin name="gazebo_ros_joint_state_publisher"
-            filename="libgazebo_ros_joint_state_publisher.so">
-            <update_rate>20</update_rate>
-            <joint_name>slider_joint</joint_name>
-            <joint_name>arm_joint</joint_name>
-        </plugin>
-    </gazebo>
-    <!-- This plugin will read a JointTrajectory message from the /set_joint_trajectory topic
-            and move the machine accordingly. It's a bit clunky but it works. -->
-    <!-- You'll probably want to add damping to the joints to stop them it flopping around.
-            e.g. <dynamics damping="10.0" friction="10.0"/> -->
-    <!-- Here's an example message to publish to test it:
-            ros2 topic pub -1 /set_joint_trajectory trajectory_msgs/msg/JointTrajectory  '{header: {frame_id: world}, joint_names: [slider_joint, arm_joint], points: [  {positions: {0.8,0.6}} ]}' -->
-    <gazebo>
-        <plugin name="gazebo_ros_joint_pose_trajectory"
-            filename="libgazebo_ros_joint_pose_trajectory.so">
-            <update_rate>2</update_rate>
-        </plugin>
-    </gazebo>
-    <!-- The next section shows an example of adding a sensor, in this case a depth camera. -->
-    <!-- Due to a quirk of how cameras work, an extra joint/link is required to create an
-            "optical frame" for the sensor. That isn't the focus for this tutorial, but you can
-            look at https://www.ros.org/reps/rep-0103.html#suffix-frames for slightly more information. -->
-    <!-- First, create the link and joint for the optical frame -->
-    <joint name="camera_optical_joint" type="fixed">
-        <origin xyz="0 0 0" rpy="-1.571 0 -1.571" />
-        <parent link="camera_link" />
-        <child link="camera_link_optical" />
-    </joint>
-    <link name="camera_link_optical"></link>
-    <!-- Add a gazebo tag for the ORIGINAL camera_link (but in the plugin we reference the optical frame so that ROS can orient things correctly) -->
-    <!-- Within the gazebo tag we have the sensor tag, and inside that there is (among other things) the camera tag with the camera parameters,
-            and the plugin tag with some extra parameters the plugin needs. -->
-    <!-- Note that although visualise is set to true, it won't actually visualise the depth camera in gazebo. To see the preview,
-            try swapping "depth" to "camera"-->
-    <gazebo reference="camera_link">
-        <sensor type="depth" name="my_camera">
-            <update_rate>20</update_rate>
-            <visualize>true</visualize>
-            <camera name="cam">
-                <horizontal_fov>1.3962634</horizontal_fov>
-                <image>
-                    <width>640</width>
-                    <height>480</height>
-                    <format>R8B8G8</format>
-                </image>
-                <clip>
-                    <near>0.02</near>
-                    <far>300</far>
-                </clip>
-                <noise>
-                    <type>gaussian</type>
-                    <mean>0.0</mean>
-                    <stddev>0.007</stddev>
-                </noise>
-            </camera>
-            <plugin name="camera_controller" filename="libgazebo_ros_camera.so">
-                <frame_name>camera_link_optical</frame_name>
-                <min_depth>0.1</min_depth>
-                <max_depth>500</max_depth>
-            </plugin>
-        </sensor>
-    </gazebo>
 </robot>

File: description/example_include.xacro (robot description, xacro)
@@ -1,5 +1,4 @@
 <?xml version="1.0"?>
 <robot xmlns:xacro="http://www.ros.org/wiki/xacro" >
-    <!-- This file is not a robot in and of itself, it just contains some useful tags that could be included in any robot -->
     <!-- Specify some colours -->
     <material name="white">
@@ -12,6 +11,4 @@
         <color rgba="0.2 0.2 1 1"/>
     </material>
-    <!-- Specify some standard inertial calculations https://en.wikipedia.org/wiki/List_of_moments_of_inertia -->
-    <!-- These make use of xacro's mathematical functionality -->
     <xacro:macro name="inertial_sphere" params="mass radius *origin">
         <inertial>

File: description/robot_core.xacro (robot description, xacro)
@@ -2,5 +2,5 @@
 <robot xmlns:xacro="http://www.ros.org/wiki/xacro"  name="robot">
     <xacro:include filename="example_include.xacro" />
-    <!-- <xacro:include filename="example_gazebo.xacro" /> -->
+    <xacro:include filename="example_gazebo.xacro" />
     <link name="world"></link>
     <!-- A simple fixed joint from our empty world link, to our base. -->
@@ -29,11 +29,11 @@
             <origin xyz="0 0 0.05" rpy="0 0 0"/>
             <geometry>
-                <box size="5 5 0.1" />
-            </geometry>
-        </collision>
-        <inertial>
-            <origin xyz="0 0 0.05" rpy="0 0 0"/>
-            <mass value="12" />
-            <inertia ixx="2.26" ixy="0.0" ixz="0.0" iyy="6.26" iyz="0.0" izz="8.5" />
+                <box size="0 0 0" />
+            </geometry>
+        </collision>
+        <inertial>
+            <origin xyz="0 0 0" rpy="0 0 0"/>
+            <mass value="10" />
+            <inertia ixx="0.01" ixy="0" ixz="0" iyy="0.01" iyz="0.0" izz="0.01" />
         </inertial>
     </link>
@@ -54,13 +54,13 @@
         </visual>
         <collision>
-            <origin xyz="2.5 2.5 0.05" rpy="0 0 0"/>
-            <geometry>
-                <box size="0.25 0.25 2" />
-            </geometry>
-        </collision>
-        <inertial>
-            <origin xyz="0 0 0.05" rpy="0 0 0"/>
-            <mass value="12" />
-            <inertia ixx="2.26" ixy="0.0" ixz="0.0" iyy="6.26" iyz="0.0" izz="8.5" />
+            <origin xyz="0 0 0" rpy="0 0 0"/>
+            <geometry>
+                <box size="0.25 0.25 2" />
+            </geometry>
+        </collision>
+        <inertial>
+            <origin xyz="0 0 0" rpy="0 0 0"/>
+            <mass value="3" />
+            <inertia ixx="0.01" ixy="0" ixz="0" iyy="0.01" iyz="0.0" izz="0.01" />
         </inertial>
     </link>
@@ -81,13 +81,13 @@
         </visual>
         <collision>
-            <origin xyz="2.5 2.5 0.05" rpy="0 0 0"/>
-            <geometry>
-                <box size="0.25 0.25 2" />
-            </geometry>
-        </collision>
-        <inertial>
-            <origin xyz="0 0 0.05" rpy="0 0 0"/>
-            <mass value="12" />
-            <inertia ixx="2.26" ixy="0.0" ixz="0.0" iyy="6.26" iyz="0.0" izz="8.5" />
+            <origin xyz="0 0 0" rpy="0 0 0"/>
+            <geometry>
+                <box size="0.25 0.25 2" />
+            </geometry>
+        </collision>
+        <inertial>
+            <origin xyz="0 0 0" rpy="0 0 0"/>
+            <mass value="3" />
+            <inertia ixx="0.01" ixy="0" ixz="0" iyy="0.01" iyz="0.0" izz="0.01" />
         </inertial>
     </link>
@@ -108,13 +108,13 @@
         </visual>
         <collision>
-            <origin xyz="2.5 2.5 0.05" rpy="0 0 0"/>
-            <geometry>
-                <box size="0.25 0.25 2" />
-            </geometry>
-        </collision>
-        <inertial>
-            <origin xyz="0 0 0.05" rpy="0 0 0"/>
-            <mass value="12" />
-            <inertia ixx="2.26" ixy="0.0" ixz="0.0" iyy="6.26" iyz="0.0" izz="8.5" />
+            <origin xyz="0 0 0" rpy="0 0 0"/>
+            <geometry>
+                <box size="0.25 0.25 2" />
+            </geometry>
+        </collision>
+        <inertial>
+            <origin xyz="0 0 0" rpy="0 0 0"/>
+            <mass value="3" />
+            <inertia ixx="0.01" ixy="0" ixz="0" iyy="0.01" iyz="0.0" izz="0.01" />
         </inertial>
     </link>
@@ -135,13 +135,13 @@
         </visual>
         <collision>
-            <origin xyz="2.5 2.5 0.05" rpy="0 0 0"/>
-            <geometry>
-                <box size="0.25 0.25 2" />
-            </geometry>
-        </collision>
-        <inertial>
-            <origin xyz="0 0 0.05" rpy="0 0 0"/>
-            <mass value="12" />
-            <inertia ixx="2.26" ixy="0.0" ixz="0.0" iyy="6.26" iyz="0.0" izz="8.5" />
+            <origin xyz="0 0 0" rpy="0 0 0"/>
+            <geometry>
+                <box size="0.25 0.25 2" />
+            </geometry>
+        </collision>
+        <inertial>
+            <origin xyz="0 0 0" rpy="0 0 0"/>
+            <mass value="3" />
+            <inertia ixx="0.01" ixy="0" ixz="0" iyy="0.01" iyz="0.0" izz="0.01" />
         </inertial>
     </link>
@@ -168,7 +168,7 @@
         </collision>
         <inertial>
-            <origin xyz="0 0 0.05" rpy="0 0 0"/>
-            <mass value="12" />
-            <inertia ixx="2.26" ixy="0.0" ixz="0.0" iyy="6.26" iyz="0.0" izz="8.5" />
+            <origin xyz="0 0 0" rpy="0 0 0"/>
+            <mass value="3" />
+            <inertia ixx="0.01" ixy="0" ixz="0" iyy="0.01" iyz="0.0" izz="0.01" />
         </inertial>
     </link>
@@ -195,7 +195,7 @@
         </collision>
         <inertial>
-            <origin xyz="0 0 0.05" rpy="0 0 0"/>
-            <mass value="12" />
-            <inertia ixx="2.26" ixy="0.0" ixz="0.0" iyy="6.26" iyz="0.0" izz="8.5" />
+            <origin xyz="0 0 0" rpy="0 0 0"/>
+            <mass value="3" />
+            <inertia ixx="0.01" ixy="0" ixz="0" iyy="0.01" iyz="0.0" izz="0.01" />
         </inertial>
     </link>
@@ -204,6 +204,7 @@
         <parent link="edge2_link"/>
         <child link="y_link"/>
-         <axis xyz="0 1 0"/>
-        <limit lower="-2.25" upper="2.25" velocity="100" effort="100"/>
+        <axis xyz="0 1 0"/>
+        <dynamics damping="5.0" friction="1.0"/>
+        <limit lower="-2.25" upper="2.25" velocity="1" effort="100"/>
     </joint>
     <link name="y_link">
@@ -218,5 +219,5 @@
         </visual>
         <collision>
-            <origin xyz="2.325 0 0" rpy="0 0 0"/>
+            <origin xyz="0 0 0" rpy="0 0 0"/>
             <geometry>
                 <box size="4.5 0.25 0.25" />
@@ -224,7 +225,7 @@
         </collision>
         <inertial>
-            <origin xyz="0 0 0.05" rpy="0 0 0"/>
-            <mass value="12" />
-            <inertia ixx="2.26" ixy="0.0" ixz="0.0" iyy="6.26" iyz="0.0" izz="8.5" />
+            <origin xyz="0 0 0" rpy="0 0 0"/>
+            <mass value="2" />
+            <inertia ixx="0.01" ixy="0" ixz="0" iyy="0.01" iyz="0.0" izz="0.01" />
         </inertial>
     </link>
@@ -233,6 +234,7 @@
         <parent link="y_link"/>
         <child link="x_link"/>
-         <axis xyz="1 0 0"/>
-        <limit lower="-2.1" upper="2.1" velocity="100" effort="100"/>
+        <axis xyz="1 0 0"/>
+        <dynamics damping="5.0" friction="1.0"/>
+        <limit lower="-2.1" upper="2.1" velocity="1" effort="100"/>
     </joint>
     <link name="x_link">
@@ -247,5 +249,5 @@
         </visual>
         <collision>
-            <origin xyz="0 0 -0.25" rpy="0 0 0"/>
+            <origin xyz="0 0 0" rpy="0 0 0"/>
             <geometry>
                 <box size="0.25 0.25 1.5" />
@@ -253,7 +255,7 @@
         </collision>
         <inertial>
-            <origin xyz="0 0 0.05" rpy="0 0 0"/>
-            <mass value="12" />
-            <inertia ixx="2.26" ixy="0.0" ixz="0.0" iyy="6.26" iyz="0.0" izz="8.5" />
+            <origin xyz="0 0 0" rpy="0 0 0"/>
+            <mass value="1" />
+            <inertia ixx="0.01" ixy="0" ixz="0" iyy="0.01" iyz="0.0" izz="0.01" />
         </inertial>
     </link>
@@ -262,6 +264,7 @@
         <parent link="x_link"/>
         <child link="z_link"/>
-         <axis xyz="0 0 1"/>
-        <limit lower="-1" upper="0.2" velocity="100" effort="100"/>
+        <axis xyz="0 0 1"/>
+        <dynamics damping="5.0" friction="1.0"/>
+        <limit lower="-1" upper="0.2" velocity="1" effort="100"/>
     </joint>
     <link name="z_link">
@@ -274,5 +277,5 @@
         </visual>
         <collision>
-            <origin xyz="0 0 -0.25" rpy="0 0 0"/>
+            <origin xyz="0 0 0" rpy="0 0 0"/>
             <geometry>
                 <box size="0.25 0.25 0.4" />
@@ -280,7 +283,7 @@
         </collision>
         <inertial>
-            <origin xyz="0 0 0.05" rpy="0 0 0"/>
-            <mass value="12" />
-            <inertia ixx="2.26" ixy="0.0" ixz="0.0" iyy="6.26" iyz="0.0" izz="8.5" />
+            <origin xyz="0 0 0" rpy="0 0 0"/>
+            <mass value="0.5" />
+            <inertia ixx="0.01" ixy="0" ixz="0" iyy="0.01" iyz="0.0" izz="0.01" />
         </inertial>
     </link>

Commit message: fix controller_managers won't loaded. because comment in xacro (URDF) not allow using special character

File: description/example_gazebo.xacro (robot description, xacro)
@@ -1,9 +1,4 @@
 <?xml version="1.0"?>
-<robot xmlns:xacro="http://www.ros.org/wiki/xacro">
-    <!-- This file demonstrates the use of some <gazebo> tags -->
-    <!-- To include it add the following line -->
-    <!-- <xacro:include filename="example_gazebo.xacro" /> -->
-    <!-- Gazebo is unable to use the same <material> tags that are already in the URDF (that RViz uses). -->
-    <!-- Instead, we need to add gazebo tags for our links that refer to Gazebo materials -->
+<robot xmlns:xacro="http://www.ros.org/wiki/xacro" name="GantBot">
     <gazebo reference="base_link">
         <material>Gazebo/Green</material>
@@ -18,5 +13,4 @@
         <material>Gazebo/Orange</material>
     </gazebo>
-    <!-- Gazebo requires the use of plugins to interact with other systems such as ROS. -->
     <ros2_control name="GazeboSystem" type="system">
         <hardware>
@@ -24,19 +18,40 @@
         </hardware>
         <joint name="x_joint">
-            <command_interface name="position" />
-            <state_interface name="position" />
+            <command_interface name="position">
+                <param name="min">-2.25</param>
+                <param name="max">2.25</param>
+            </command_interface>
+            <state_interface name="position">
+                <param name="initial_value">0.0</param>
+            </state_interface>
+            <state_interface name="velocity"/>
+            <state_interface name="effort"/>
         </joint>
         <joint name="y_joint">
-            <command_interface name="position" />
-            <state_interface name="position" />
+            <command_interface name="position">
+                <param name="min">-2.1</param>
+                <param name="max">2.1</param>
+            </command_interface>
+            <state_interface name="position">
+                <param name="initial_value">-0.5</param>
+            </state_interface>
+            <state_interface name="velocity"/>
+            <state_interface name="effort"/>
         </joint>
         <joint name="z_joint">
-            <command_interface name="position" />
-            <state_interface name="position" />
+            <command_interface name="position">
+                <param name="min">-1</param>
+                <param name="max">0.2</param>
+            </command_interface>
+            <state_interface name="position">
+                <param name="initial_value">-0.5</param>
+            </state_interface>
+            <state_interface name="velocity"/>
+            <state_interface name="effort"/>
         </joint>
     </ros2_control>
     <gazebo>
         <plugin name="gazebo_ros2_control" filename="libgazebo_ros2_control.so">
-            <parameter> $find(GantBot)/config/gantry_controller.yaml </parameter>
+            <parameters>$(find GantBot)/config/gantry_controller.yaml</parameters>
         </plugin>
     </gazebo>

File: description/example_include.xacro (robot description, xacro)
@@ -1,5 +1,4 @@
 <?xml version="1.0"?>
-<robot xmlns:xacro="http://www.ros.org/wiki/xacro" >
-    <!-- Specify some colours -->
+<robot xmlns:xacro="http://www.ros.org/wiki/xacro" name="GantBot">
     <material name="white">
         <color rgba="1 1 1 1"/>

File: description/robot.urdf.xacro (robot description, xacro)
@@ -1,6 +1,6 @@
 <?xml version="1.0"?>
-<robot xmlns:xacro="http://www.ros.org/wiki/xacro"  name="robot">
+<robot xmlns:xacro="http://www.ros.org/wiki/xacro" name="GantBot">
     <xacro:arg name="use_ros2_control" default="true"/>
-    <xacro:arg name="sim_mode" default="false"/>
+    <xacro:arg name="sim_mode" default="true"/>
     <xacro:include filename="robot_core.xacro" />
 </robot>

File: description/robot_core.xacro (robot description, xacro)
@@ -1,9 +1,7 @@
 <?xml version="1.0"?>
-<robot xmlns:xacro="http://www.ros.org/wiki/xacro"  name="robot">
+<robot xmlns:xacro="http://www.ros.org/wiki/xacro" name="GantBot">
     <xacro:include filename="example_include.xacro" />
     <xacro:include filename="example_gazebo.xacro" />
     <link name="world"></link>
-    <!-- A simple fixed joint from our empty world link, to our base. -->
-    <!-- The base origin is offset from the world origin. -->
     <joint name="base_joint" type="fixed">
         <origin xyz="1.5 1.0 0" rpy="0 0 0"/>
@@ -12,9 +10,4 @@
         <dynamics damping="1000000" friction="10000000"/>
     </joint>
-    <!-- base_link is a large rectangular plate. Some things to note: -->
-    <!-- - We set the visual origin Z to half the box height, so that the link origin sits at the bottom of the box -->
-    <!-- - We set the collision to be identical to the visual -->
-    <!-- - We specified the colour manually (but still need to enter a name) -->
-    <!-- - We specified all the inertial parameters manually -->
     <link name="base_link">
         <visual>
@@ -268,5 +261,5 @@
             <origin xyz="0 0 -0.6" rpy="0 0 0"/>
             <geometry>
-                <box size="0.25 0.25 0.4" />
+                <box size="0.25 0.25 0.4"/>
             </geometry>
         </collision>
